Commit message: The husky mesh for the top plate added, as well as the top bracket (the original model, mesh needs refinement). Head -> body transform should now be correct.

File: software/models/husky_description/model.urdf (robot description, URDF)
Before this commit: robot husky, 14 links, 13 joints
Links:
- removed link top_plate_link
- added link 300Arch; visual mesh filename=package://husky_description/meshes/300Arch.STL
- added link topPlate; visual mesh filename=package://husky_description/meshes/short_top_plate.STL
Joints:
- removed joint top_plate_joint
- added joint base_link_to_topPlate: type fixed, parent base_link, child topPlate, origin xyz=0.02 0.0 0.2503 rpy=0.0 0.0 0.0
- added joint topPlate_to_300Arch: type fixed, parent topPlate, child 300Arch, origin xyz=-0.28 0.0 0.3 rpy=0.0 0.0 3.14159

Commit message: Added signal scope scripts for the IMU preview of the husky and the standalone one. Modified the URDF to fix the IMU orientation.

File: software/models/husky_description/model.urdf (robot description, URDF)
Before this commit: robot husky, 15 links, 14 joints
Joints:
- joint imu_joint: origin xyz=0.19 0 0.149 rpy=0 -1.5708 3.1416 -> xyz=0.19 0 0.149 rpy=0 1.5705 0
