Commit message: URDF: transformation for asus xtion camera frame "head_xtion_link"

File: software/models/val_description/urdf/valkyrie_sim.urdf (robot description, URDF)
Before this commit: robot valkyrie, 84 links, 83 joints
Links:
- added link head_xtion_link
Joints:
- added joint head_xtion_joint: type fixed, parent head, child head_xtion_link, origin xyz=0.02 -0.025 -0.05 rpy=1.082104136 0.0 1.570796327
