Commit message: Add dual arm husky simple mesh model

File: software/models/dual_arm_husky_description/urdf/dual_arm_husky_original.urdf (robot description, URDF)
Before this commit: robot husky, 124 links, 123 joints
Links:
- link base_laser: geometry collision box size=0.105 0.1 0.1; visual mesh filename=package://dual_arm_husky_description/meshes/sick-lms1xx.dae
- link base_link: geometry collision box size=0.78992 0.5709 0.12375; collision box size=0.9874 0.5709 0.12375
- link front_bumper_link: geometry visual mesh filename=package://dual_arm_husky_description/meshes/bumper.dae
- link front_left_wheel_link: geometry collision cylinder length=0.1143 radius=0.17775; visual mesh filename=package://dual_arm_husky_description/meshes/wheel.dae
- link front_right_wheel_link: geometry collision cylinder length=0.1143 radius=0.17775; visual mesh filename=package://dual_arm_husky_description/meshes/wheel.dae
- link l_ur5_arm_base_link: geometry collision mesh filename=package://ur_description/meshes/ur5/collision/base.stl; visual mesh filename=package://ur_description/meshes/ur5/visual/base.dae
- link l_ur5_arm_forearm_link: geometry collision mesh filename=package://ur_description/meshes/ur5/collision/forearm.stl; visual mesh filename=package://ur_description/meshes/ur5/visual/forearm.dae
- link l_ur5_arm_shoulder_link: geometry collision mesh filename=package://ur_description/meshes/ur5/collision/shoulder.stl; visual mesh filename=package://ur_description/meshes/ur5/visual/shoulder.dae
- link l_ur5_arm_upper_arm_link: geometry collision mesh filename=package://ur_description/meshes/ur5/collision/upperarm.stl; visual mesh filename=package://ur_description/meshes/ur5/visual/upperarm.dae
- link l_ur5_arm_wrist_1_link: geometry collision mesh filename=package://ur_description/meshes/ur5/collision/wrist1.stl; visual mesh filename=package://ur_description/meshes/ur5/visual/wrist1.dae
- link l_ur5_arm_wrist_2_link: geometry collision mesh filename=package://ur_description/meshes/ur5/collision/wrist2.stl; visual mesh filename=package://ur_description/meshes/ur5/visual/wrist2.dae
- link l_ur5_arm_wrist_3_link: geometry collision mesh filename=package://ur_description/meshes/ur5/collision/wrist3.stl; visual mesh filename=package://ur_description/meshes/ur5/visual/wrist3.dae
- link r_ur5_arm_base_link: geometry collision mesh filename=package://ur_description/meshes/ur5/collision/base.stl; visual mesh filename=package://ur_description/meshes/ur5/visual/base.dae
- link r_ur5_arm_forearm_link: geometry collision mesh filename=package://ur_description/meshes/ur5/collision/forearm.stl; visual mesh filename=package://ur_description/meshes/ur5/visual/forearm.dae
- link r_ur5_arm_shoulder_link: geometry collision mesh filename=package://ur_description/meshes/ur5/collision/shoulder.stl; visual mesh filename=package://ur_description/meshes/ur5/visual/shoulder.dae
- link r_ur5_arm_upper_arm_link: geometry collision mesh filename=package://ur_description/meshes/ur5/collision/upperarm.stl; visual mesh filename=package://ur_description/meshes/ur5/visual/upperarm.dae
- link r_ur5_arm_wrist_1_link: geometry collision mesh filename=package://ur_description/meshes/ur5/collision/wrist1.stl; visual mesh filename=package://ur_description/meshes/ur5/visual/wrist1.dae
- link r_ur5_arm_wrist_2_link: geometry collision mesh filename=package://ur_description/meshes/ur5/collision/wrist2.stl; visual mesh filename=package://ur_description/meshes/ur5/visual/wrist2.dae
- link r_ur5_arm_wrist_3_link: geometry collision mesh filename=package://ur_description/meshes/ur5/collision/wrist3.stl; visual mesh filename=package://ur_description/meshes/ur5/visual/wrist3.dae
- link rear_bumper_link: geometry visual mesh filename=package://dual_arm_husky_description/meshes/bumper.dae
- link rear_left_wheel_link: geometry collision cylinder length=0.1143 radius=0.17775; visual mesh filename=package://dual_arm_husky_description/meshes/wheel.dae
- link rear_right_wheel_link: geometry collision cylinder length=0.1143 radius=0.17775; visual mesh filename=package://dual_arm_husky_description/meshes/wheel.dae
- link top_chassis_link: geometry visual mesh filename=package://dual_arm_husky_description/meshes/top_chassis.dae
