Commit message: Add flir-ptu-simple.stl

File: software/models/dual_arm_husky_description/urdf/dual_arm_husky.urdf (robot description, URDF)
Before this commit: robot husky, 124 links, 123 joints
Links:
- link husky_ptu_pan_link: geometry collision box size=0.045 0.065 0.044; collision box size=0.046 0.044 0.044
- link husky_ptu_tilt_link: geometry collision box size=0.045 0.065 0.044; collision box size=0.046 0.044 0.044

Commit message: rm lms1xx and move meshes into dual_arm_husky_description

File: software/models/dual_arm_husky_description/urdf/dual_arm_husky.urdf (robot description, URDF)
Before this commit: robot husky, 124 links, 123 joints
Links:
- link base_laser: geometry collision box size=0.105 0.1 0.1; visual mesh filename=package://dual_arm_husky_description/meshes/sick-lms1xx.dae

File: software/models/dual_arm_husky_description/urdf/dual_arm_husky_drake.urdf (robot description, URDF)
Before this commit: robot husky, 39 links, 38 joints
Links:
- link base_laser: geometry collision box size=0.105 0.1 0.1; visual mesh filename=package://dual_arm_husky_description/meshes/sick-lms1xx.dae

Commit message: Move fts300 sensor into dual_arm_husky_description

File: software/models/dual_arm_husky_description/urdf/dual_arm_husky.urdf (robot description, URDF)
Before this commit: robot husky, 124 links, 123 joints
Links:
- link l_robotiq_fts300_fts_robotside: geometry collision mesh filename=package://dual_arm_husky_description/meshes/collision/robot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; visual mesh filename=package://dual_arm_husky_description/meshes/visual/robotiq_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
- link r_robotiq_fts300_fts_robotside: geometry collision mesh filename=package://dual_arm_husky_description/meshes/collision/robot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; visual mesh filename=package://dual_arm_husky_description/meshes/visual/robotiq_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

File: software/models/dual_arm_husky_description/urdf/dual_arm_husky_drake.urdf (robot description, URDF)
Before this commit: robot husky, 39 links, 38 joints
Links:
- link l_robotiq_fts300_fts_robotside: geometry collision mesh filename=package://dual_arm_husky_description/meshes/collision/robot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; visual mesh filename=package://dual_arm_husky_description/meshes/visual/robotiq_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
- link r_robotiq_fts300_fts_robotside: geometry collision mesh filename=package://dual_arm_husky_description/meshes/collision/robot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; visual mesh filename=package://dual_arm_husky_description/meshes/visual/robotiq_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

Commit message: Activate bumblebee in current URDF and add mesh

File: software/models/dual_arm_husky_description/urdf/dual_arm_husky.urdf (robot description, URDF)
Before this commit: robot husky, 124 links, 123 joints
Links:
- added link bumblebee2, mass 0.342; collision box size=0.04740 0.157 0.036; visual mesh filename=package://dual_arm_husky_description/meshes/pointgrey_bumbl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
- added link bumblebee2_optical, mass 1E-5
Joints:
- added joint bumblebee2_mount_joint: type fixed, parent husky_ptu_mount_link, child bumblebee2, origin xyz=-0.079 0.02 -0.10 rpy=3.14 1.57 0
- added joint bumblebee2_optical_joint: type fixed, parent bumblebee2, child bumblebee2_optical, origin xyz=0 0 0 rpy=-1.570796 0 -1.570796

Commit message: Revert left_/l_ and right_/r_ for finger to be consistent with ROS

File: software/models/dual_arm_husky_description/urdf/dual_arm_husky.urdf (robot description, URDF)
Before this commit: robot husky, 126 links, 125 joints
Links:
- added link l_palm, mass 1.3; collision box size=0.1 0.1 0.1; visual mesh filename=package://robotiq_hand_description/meshes/s-model_articulat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
- added link r_palm, mass 1.3; collision box size=0.1 0.1 0.1; visual mesh filename=package://robotiq_hand_description/meshes/s-model_articulat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
- link left_palm: mass 1.3 -> None; geometry 
- link right_palm: mass 1.3 -> None; geometry 
Joints:
- removed joint left_palm_finger_1_joint
- removed joint left_palm_finger_2_joint
- removed joint left_palm_finger_middle_joint
- removed joint right_palm_finger_1_joint
- removed joint right_palm_finger_2_joint
- removed joint right_palm_finger_middle_joint
- added joint l_palm_finger_1_joint: type revolute, parent l_palm, child l_finger_1_link_0, origin xyz=-0.0455 0.0214 0.036 rpy=0 3.1416 -1.57, axis 0 1 0, limit lower=-0.2967 upper=0.2967 effort=60 velocity=-1
- added joint l_palm_finger_2_joint: type revolute, parent l_palm, child l_finger_2_link_0, origin xyz=-0.0455 0.0214 -0.036 rpy=0 3.1416 -1.57, axis 0 1 0, limit lower=-0.2967 upper=0.2967 effort=60 velocity=-1
- added joint l_palm_finger_middle_joint: type revolute, parent l_palm, child l_finger_middle_link_0, origin xyz=0.0455 0.0214 0 rpy=0 0 1.57, axis 0 1 0, limit lower=0 upper=0 effort=60 velocity=-1
- added joint l_palm_to_left_palm_fixed_joint: type fixed, parent l_palm, child left_palm, origin xyz=0 0 0 rpy=0 0 0
- added joint r_palm_finger_1_joint: type revolute, parent r_palm, child r_finger_1_link_0, origin xyz=-0.0455 0.0214 0.036 rpy=0 3.1416 -1.57, axis 0 1 0, limit lower=-0.2967 upper=0.2967 effort=60 velocity=-1
- added joint r_palm_finger_2_joint: type revolute, parent r_palm, child r_finger_2_link_0, origin xyz=-0.0455 0.0214 -0.036 rpy=0 3.1416 -1.57, axis 0 1 0, limit lower=-0.2967 upper=0.2967 effort=60 velocity=-1
- added joint r_palm_finger_middle_joint: type revolute, parent r_palm, child r_finger_middle_link_0, origin xyz=0.0455 0.0214 0 rpy=0 0 1.57, axis 0 1 0, limit lower=0 upper=0 effort=60 velocity=-1
- added joint r_palm_to_right_palm_fixed_joint: type fixed, parent r_palm, child right_palm, origin xyz=0 0 0 rpy=0 0 0
- joint l_robotiq_hand_joint: child left_palm -> l_palm
- joint r_robotiq_hand_joint: child right_palm -> r_palm

File: software/models/dual_arm_husky_description/urdf/dual_arm_husky_original.urdf (robot description, URDF)
Before this commit: robot husky, 126 links, 125 joints
Links:
- added link l_palm, mass 1.3; collision box size=0.1 0.1 0.1; visual mesh filename=package://robotiq_hand_description/meshes/s-model_articulat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
- added link r_palm, mass 1.3; collision box size=0.1 0.1 0.1; visual mesh filename=package://robotiq_hand_description/meshes/s-model_articulat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
- link left_palm: mass 1.3 -> None; geometry 
- link right_palm: mass 1.3 -> None; geometry 
Joints:
- removed joint left_palm_finger_1_joint
- removed joint left_palm_finger_2_joint
- removed joint left_palm_finger_middle_joint
- removed joint right_palm_finger_1_joint
- removed joint right_palm_finger_2_joint
- removed joint right_palm_finger_middle_joint
- added joint l_palm_finger_1_joint: type revolute, parent l_palm, child l_finger_1_link_0, origin xyz=-0.0455 0.0214 0.036 rpy=0 3.1416 -1.57, axis 0 1 0, limit lower=-0.2967 upper=0.2967 effort=60 velocity=-1
- added joint l_palm_finger_2_joint: type revolute, parent l_palm, child l_finger_2_link_0, origin xyz=-0.0455 0.0214 -0.036 rpy=0 3.1416 -1.57, axis 0 1 0, limit lower=-0.2967 upper=0.2967 effort=60 velocity=-1
- added joint l_palm_finger_middle_joint: type revolute, parent l_palm, child l_finger_middle_link_0, origin xyz=0.0455 0.0214 0 rpy=0 0 1.57, axis 0 1 0, limit lower=0 upper=0 effort=60 velocity=-1
- added joint l_palm_to_left_palm_fixed_joint: type fixed, parent l_palm, child left_palm, origin xyz=0 0 0 rpy=0 0 0
- added joint r_palm_finger_1_joint: type revolute, parent r_palm, child r_finger_1_link_0, origin xyz=-0.0455 0.0214 0.036 rpy=0 3.1416 -1.57, axis 0 1 0, limit lower=-0.2967 upper=0.2967 effort=60 velocity=-1
- added joint r_palm_finger_2_joint: type revolute, parent r_palm, child r_finger_2_link_0, origin xyz=-0.0455 0.0214 -0.036 rpy=0 3.1416 -1.57, axis 0 1 0, limit lower=-0.2967 upper=0.2967 effort=60 velocity=-1
- added joint r_palm_finger_middle_joint: type revolute, parent r_palm, child r_finger_middle_link_0, origin xyz=0.0455 0.0214 0 rpy=0 0 1.57, axis 0 1 0, limit lower=0 upper=0 effort=60 velocity=-1
- added joint r_palm_to_right_palm_fixed_joint: type fixed, parent r_palm, child right_palm, origin xyz=0 0 0 rpy=0 0 0
- joint l_robotiq_hand_joint: child left_palm -> l_palm
- joint r_robotiq_hand_joint: child right_palm -> r_palm

Commit message: Fix PTU axes

File: software/models/dual_arm_husky_description/urdf/dual_arm_husky.urdf (robot description, URDF)
Before this commit: robot husky, 128 links, 127 joints
Joints:
- joint bumblebee2_mount_joint: origin xyz=-0.079 0.02 -0.10 rpy=3.14 1.57 0 -> xyz=0 0 0.00 rpy=0 0 0
- joint husky_ptu_joint: origin xyz=0.365 0 0.221 rpy=0 1.57 3.14 -> xyz=0.365 0 0.221 rpy=0 0 0

File: software/models/dual_arm_husky_description/urdf/dual_arm_husky_original.urdf (robot description, URDF)
Before this commit: robot husky, 128 links, 127 joints
Joints:
- joint bumblebee2_mount_joint: origin xyz=-0.079 0.02 -0.10 rpy=3.14 1.57 0 -> xyz=0 0 0.00 rpy=0 0 0
- joint husky_ptu_joint: origin xyz=0.365 0 0.221 rpy=0 1.57 3.14 -> xyz=0.365 0 0.19876 rpy=0 0 0

Commit message: Fix Robotiq mount z-offset

File: software/models/dual_arm_husky_description/urdf/dual_arm_husky.urdf (robot description, URDF)
Before this commit: robot dual_arm_husky, 128 links, 127 joints
Joints:
- joint l_robotiq_hand_joint: origin xyz=0 0 0 rpy=1.57 0 0 -> xyz=0 0 0.05398 rpy=1.57 0 0
- joint r_robotiq_hand_joint: origin xyz=0 0 0 rpy=1.57 0 0 -> xyz=0 0 0.05398 rpy=1.57 0 0

File: software/models/dual_arm_husky_description/urdf/dual_arm_husky_original.urdf (robot description, URDF)
Before this commit: robot dual_arm_husky, 128 links, 127 joints
Joints:
- joint l_robotiq_hand_joint: origin xyz=0 0 0 rpy=1.57 0 0 -> xyz=0 0 0.05398 rpy=1.57 0 0
- joint r_robotiq_hand_joint: origin xyz=0 0 0 rpy=1.57 0 0 -> xyz=0 0 0.05398 rpy=1.57 0 0

Commit message: Fix hand orientation approximately by eye in URDFs

File: software/models/dual_arm_husky_description/urdf/dual_arm_husky.urdf (robot description, URDF)
Before this commit: robot dual_arm_husky, 128 links, 127 joints
Joints:
- joint l_robotiq_hand_joint: origin xyz=0 0 0.05398 rpy=1.57 0 0 -> xyz=0 0 0.05398 rpy=1.57 0 1.0
- joint r_robotiq_hand_joint: origin xyz=0 0 0.05398 rpy=1.57 0 0 -> xyz=0 0 0.05398 rpy=1.57 0 2.355

File: software/models/dual_arm_husky_description/urdf/dual_arm_husky_original.urdf (robot description, URDF)
Before this commit: robot dual_arm_husky, 128 links, 127 joints
Joints:
- joint l_robotiq_hand_joint: origin xyz=0 0 0.05398 rpy=1.57 0 0 -> xyz=0 0 0.05398 rpy=1.57 0 1.0
- joint r_robotiq_hand_joint: origin xyz=0 0 0.05398 rpy=1.57 0 0 -> xyz=0 0 0.05398 rpy=1.57 0 2.355

Commit message: Fix IMU joint in URDFs

File: software/models/dual_arm_husky_description/urdf/dual_arm_husky.urdf (robot description, URDF)
Before this commit: robot dual_arm_husky, 128 links, 127 joints
Joints:
- joint imu_joint: origin xyz=0.19 0 0.149 rpy=0 -1.5708 3.1416 -> xyz=0.19 0 0.149 rpy=-1.5708 0 0

File: software/models/dual_arm_husky_description/urdf/dual_arm_husky_drake.urdf (robot description, URDF)
Before this commit: robot dual_arm_husky, 39 links, 38 joints
Joints:
- joint imu_joint: origin xyz=0.19 0 0.149 rpy=0 -1.5708 3.1416 -> xyz=0.19 0 0.149 rpy=-1.5708 0 0

File: software/models/dual_arm_husky_description/urdf/dual_arm_husky_original.urdf (robot description, URDF)
Before this commit: robot dual_arm_husky, 128 links, 127 joints
Joints:
- joint imu_joint: origin xyz=0.19 0 0.149 rpy=0 -1.5708 3.1416 -> xyz=0.19 0 0.149 rpy=-1.5708 0 0

Commit message: Fix PTU mount offsets (another Clearpath integration mishap)

File: software/models/dual_arm_husky_description/urdf/dual_arm_husky.urdf (robot description, URDF)
Before this commit: robot dual_arm_husky, 128 links, 127 joints
Joints:
- joint bumblebee2_mount_joint: origin xyz=0 0 0.00 rpy=0 0 0 -> xyz=0 0 0.02224 rpy=0 0 0
- joint husky_ptu_joint: origin xyz=0.365 0 0.221 rpy=0 0 0 -> xyz=0.345 0.010414 0.19876 rpy=0 0 0

File: software/models/dual_arm_husky_description/urdf/dual_arm_husky_original.urdf (robot description, URDF)
Before this commit: robot dual_arm_husky, 128 links, 127 joints
Joints:
- joint bumblebee2_mount_joint: origin xyz=0 0 0.00 rpy=0 0 0 -> xyz=0 0 0.02224 rpy=0 0 0
- joint husky_ptu_joint: origin xyz=0.365 0 0.19876 rpy=0 0 0 -> xyz=0.345 0.010414 0.19876 rpy=0 0 0

Commit message: Add Fixed Xtion Mount to URDFs

File: software/models/dual_arm_husky_description/urdf/dual_arm_husky.urdf (robot description, URDF)
Before this commit: robot dual_arm_husky, 128 links, 127 joints
Links:
- added link fixed_xtion_mount; collision cylinder length=0.82 radius=0.06; visual cylinder length=0.82 radius=0.06
Joints:
- added joint fixed_xtion_mount_joint: type fixed, parent dual_arm_bulkhead_link, child fixed_xtion_mount, origin xyz=-.24 0 .605 rpy=0 0 0

File: software/models/dual_arm_husky_description/urdf/dual_arm_husky_drake.urdf (robot description, URDF)
Before this commit: robot dual_arm_husky, 39 links, 38 joints
Links:
- added link fixed_xtion_mount; collision cylinder length=0.82 radius=0.06; visual cylinder length=0.82 radius=0.06
Joints:
- added joint fixed_xtion_mount_joint: type fixed, parent dual_arm_bulkhead_link, child fixed_xtion_mount, origin xyz=-.24 0 .605 rpy=0 0 0

File: software/models/dual_arm_husky_description/urdf/dual_arm_husky_original.urdf (robot description, URDF)
Before this commit: robot dual_arm_husky, 128 links, 127 joints
Links:
- added link fixed_xtion_mount; collision cylinder length=0.82 radius=0.06; visual cylinder length=0.82 radius=0.06
Joints:
- added joint fixed_xtion_mount_joint: type fixed, parent dual_arm_bulkhead_link, child fixed_xtion_mount, origin xyz=-.24 0 .605 rpy=0 0 0
