Commit message: add palm links to drake model

File: software/models/dual_arm_husky_description/urdf/dual_arm_husky_drake.urdf (robot description, URDF)
Before this commit: robot dual_arm_husky, 40 links, 39 joints
Links:
- added link l_palm
- added link left_palm; collision cylinder length=0.3 radius=0.1; visual cylinder length=0.3 radius=0.1
- added link r_palm
- added link right_palm; collision cylinder length=0.3 radius=0.1; visual cylinder length=0.3 radius=0.1
Joints:
- added joint l_palm_to_left_palm_fixed_joint: type fixed, parent l_palm, child left_palm, origin xyz=0 0 0 rpy=0 0 0
- added joint l_robotiq_hand_joint: type fixed, parent l_robotiq_fts300_fts_toolside, child l_palm, origin xyz=0 0 0.05398 rpy=1.57 0 1.0
- added joint r_palm_to_right_palm_fixed_joint: type fixed, parent r_palm, child right_palm, origin xyz=0 0 0 rpy=0 0 0
- added joint r_robotiq_hand_joint: type fixed, parent r_robotiq_fts300_fts_toolside, child r_palm, origin xyz=0 0 0.05398 rpy=1.57 0 2.355
